File: buck.sch (KiCad schematic (older format))
At the start: 12 parts, among them U1 AP63205

Commit message: Add fiducials, fix aesthetics in schematics
Parts:
- D8: Manufacturer (none) -> ON Semiconductor; Part Number (none) -> MBRS260T3G
- F1: Manufacturer (none) -> Bel Fuse; Part Number (none) -> 0ZCG0075BF2B
Other:
- note added: "Ihold = 750mA\nItrip = 1500mA"
- note removed: "Channel 1 is connected to a buck converter \nto provide 5V for the Feather.\nDisconnect J1 jumper if Feather has external power."
- note removed: "Disconnect the jumper\nif Feather is powered from USB,\nto prevent back-powering."
Changed lines of the file:
@@
 encoding utf-8
 Sheet 5 6
-Title ""
+Title "Tougher INA3221 Power Meter"
 Date ""
 Rev ""
-Comp ""
+Comp "Beast Devices"
 Comment1 ""
 Comment2 ""
@@
 Wire Wire Line
 	4750 3550 4750 3650
-Text Notes 6800 1800 0    50   ~ 0
-Disconnect the jumper\nif Feather is powered from USB,\nto prevent back-powering.
 Connection ~ 7600 3400
 Wire Wire Line
 	7600 3400 7950 3400
-Text Notes 4150 2000 0    50   ~ 0
-Channel 1 is connected to a buck converter \nto provide 5V for the Feather.\nDisconnect J1 jumper if Feather has external power.
 $Comp
 L Device:C_Small C2
@@
 AR Path="/5F5FC933" Ref="D?"  Part="1"
 AR Path="/5F5E3585/5F5FC933" Ref="D8"  Part="1"
-F 0 "D8" H 3100 3033 50  0000 C CNN
-F 1 "D_Schottky" H 3100 3124 50  0000 C CNN
+F 0 "D8" H 3100 3150 50  0000 C CNN
+F 1 "D_Schottky" H 3100 3124 50  0001 C CNN
 F 2 "Diode_SMD:D_SMB" H 3100 3250 50  0001 C CNN
 F 3 "~" H 3100 3250 50  0001 C CNN
+F 4 "MBRS260T3G" H 3100 3350 50  0000 C CNN "Part Number"
+F 5 "ON Semiconductor" H 3100 3250 50  0001 C CNN "Manufacturer"
 	1    3100 3250
 	-1   0    0    1
@@
 U 1 1 5F629EE9
 P 9000 3400
-F 0 "F1" V 8775 3400 50  0000 C CNN
-F 1 "0ZCG0075BF2B" V 8866 3400 50  0000 C CNN
+F 0 "F1" V 8900 3400 50  0000 C CNN
+F 1 "0ZCG0075BF2B" V 9150 3400 50  0000 C CNN
 F 2 "Fuse:Fuse_1812_4532Metric" H 9050 3200 50  0001 L CNN
 F 3 "https://www.mouser.se/datasheet/2/643/0ZCG_Nov2016-1132141.pdf" H 9000 3400 50  0001 C CNN
+F 4 "0ZCG0075BF2B" V 9000 3400 50  0001 C CNN "Part Number"
+F 5 "Bel Fuse" V 9000 3400 50  0001 C CNN "Manufacturer"
 	1    9000 3400
 	0    1    1    0
@@
 Wire Wire Line
 	8300 3400 8850 3400
+Text Notes 8700 3200 0    50   ~ 0
+Ihold = 750mA\nItrip = 1500mA
 $EndSCHEMATC

Commit message: Add manufacturers, part numbers, and supplier links
Parts:
- C2, C21: Distributor Link (none) -> https://www.digikey.se/product-detail/en/taiyo-yuden/GMK325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; Manufacturer (none) -> Taiyo Yuden; Part Number (none) -> GMK325BJ226MM-T
- C22, C3: Distributor Link (none) -> https://www.digikey.se/product-detail/en/murata-electronics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; Manufacturer (none) -> Murata Electronics; Part Number (none) -> GRM319R6YA106KA12D
- C23, C5, C6: Distributor Link (none) -> https://www.digikey.se/product-detail/en/murata-electronics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; Manufacturer (none) -> Murata Electronics; Part Number (none) -> GRM21BR61A226ME51L
- C4: footprint Resistor_SMD:R_0603_1608Metric -> Capacitor_SMD:C_0603_1608Metric; Voltage (none) -> 50V
- D8: Distributor Link (none) -> https://www.digikey.se/product-detail/en/on-semiconductor/M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
- F1: Distributor Link (none) -> https://www.digikey.se/product-detail/en/bel-fuse-inc/0ZCG0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
- L1: Distributor Link (none) -> https://www.digikey.se/product-detail/en/bourns-inc/SRR4828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; Manufacturer (none) -> Bourns Inc.
- U1: Distributor Link (none) -> https://www.digikey.se/product-detail/en/diodes-incorporate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; Manufacturer (none) -> Diodes Incorporated; Part Number (none) -> AP63205WU-7
Changed lines of the file:
@@
 F 2 "Package_TO_SOT_SMD:TSOT-23-6" H 7450 2900 50  0001 C CNN
 F 3 "https://www.mouser.se/datasheet/2/115/AP63200-AP63201-AP63203-AP63205-1525010.pdf" H 7450 2900 50  0001 C CNN
+F 4 "https://www.digikey.se/product-detail/en/diodes-incorporated/AP63205WU-7/AP63205WU-7DICT-ND/9858428" H 5600 3400 50  0001 C CNN "Distributor Link"
+F 5 "Diodes Incorporated" H 5600 3400 50  0001 C CNN "Manufacturer"
+F 6 "AP63205WU-7" H 5600 3400 50  0001 C CNN "Part Number"
 	1    5600 3400
 	1    0    0    -1
@@
 F 0 "C4" V 6150 3050 50  0000 L CNN
 F 1 "100n" V 6150 3300 50  0000 L CNN
-F 2 "Resistor_SMD:R_0603_1608Metric" H 6200 3250 50  0001 C CNN
+F 2 "Capacitor_SMD:C_0603_1608Metric" H 6200 3250 50  0001 C CNN
 F 3 "~" H 6200 3250 50  0001 C CNN
+F 4 "50V" H 6200 3250 50  0001 C CNN "Voltage"
 	1    6200 3250
 	0    1    1    0
@@
 F 3 "~" H 4750 3450 50  0001 C CNN
 F 4 "35V" H 4500 3550 50  0000 L CNN "Voltage"
+F 5 "https://www.digikey.se/product-detail/en/murata-electronics/GRM319R6YA106KA12D/490-9964-1-ND/5026458" H 4750 3450 50  0001 C CNN "Distributor Link"
+F 6 "Murata Electronics" H 4750 3450 50  0001 C CNN "Manufacturer"
+F 7 "GRM319R6YA106KA12D" H 4750 3450 50  0001 C CNN "Part Number"
 	1    4750 3450
 	-1   0    0    1
@@
 F 3 "~" H 7600 3700 50  0001 C CNN
 F 4 "10V" H 7350 3800 50  0000 L CNN "Voltage"
+F 5 "https://www.digikey.se/product-detail/en/murata-electronics/GRM21BR61A226ME51L/490-10511-1-ND/5026441" H 7600 3700 50  0001 C CNN "Distributor Link"
+F 6 "Murata Electronics" H 7600 3700 50  0001 C CNN "Manufacturer"
+F 7 "GRM21BR61A226ME51L" H 7600 3700 50  0001 C CNN "Part Number"
 	1    7600 3700
 	-1   0    0    1
@@
 F 3 "~" H 7950 3700 50  0001 C CNN
 F 4 "10V" H 7700 3800 50  0000 L CNN "Voltage"
+F 5 "https://www.digikey.se/product-detail/en/murata-electronics/GRM21BR61A226ME51L/490-10511-1-ND/5026441" H 7950 3700 50  0001 C CNN "Distributor Link"
+F 6 "Murata Electronics" H 7950 3700 50  0001 C CNN "Manufacturer"
+F 7 "GRM21BR61A226ME51L" H 7950 3700 50  0001 C CNN "Part Number"
 	1    7950 3700
 	-1   0    0    1
@@
 F 3 "https://www.bourns.com/docs/Product-Datasheets/SRR4828A.pdf" H 6700 3400 50  0001 C CNN
 F 4 "SRR4828A-4R7Y" V 6600 3400 50  0000 C CNN "Part Number"
+F 5 "https://www.digikey.se/product-detail/en/bourns-inc/SRR4828A-4R7Y/SRR4828A-4R7YCT-ND/7556072" H 6700 3400 50  0001 C CNN "Distributor Link"
+F 6 "Bourns Inc." H 6700 3400 50  0001 C CNN "Manufacturer"
 	1    6700 3400
 	0    -1   -1   0
@@
 F 3 "~" H 3950 3450 50  0001 C CNN
 F 4 "35V" H 3700 3550 50  0000 L CNN "Voltage"
+F 5 "https://www.digikey.se/product-detail/en/taiyo-yuden/GMK325BJ226MM-T/587-6141-1-ND/8619544" H 3950 3450 50  0001 C CNN "Distributor Link"
+F 6 "Taiyo Yuden" H 3950 3450 50  0001 C CNN "Manufacturer"
+F 7 "GMK325BJ226MM-T" H 3950 3450 50  0001 C CNN "Part Number"
 	1    3950 3450
 	-1   0    0    1
@@
 F 4 "MBRS260T3G" H 3100 3350 50  0000 C CNN "Part Number"
 F 5 "ON Semiconductor" H 3100 3250 50  0001 C CNN "Manufacturer"
+F 6 "https://www.digikey.se/product-detail/en/on-semiconductor/MBRS260T3G/MBRS260T3GOSCT-ND/920613" H 3100 3250 50  0001 C CNN "Distributor Link"
 	1    3100 3250
 	-1   0    0    1
@@
 F 4 "0ZCG0075BF2B" V 9000 3400 50  0001 C CNN "Part Number"
 F 5 "Bel Fuse" V 9000 3400 50  0001 C CNN "Manufacturer"
+F 6 "https://www.digikey.se/product-detail/en/bel-fuse-inc/0ZCG0075BF2B/507-1765-1-ND/4156153" H 9000 3400 50  0001 C CNN "Distributor Link"
 	1    9000 3400
 	0    1    1    0
@@
 F 3 "~" H 3600 3450 50  0001 C CNN
 F 4 "35V" H 3350 3550 50  0000 L CNN "Voltage"
+F 5 "https://www.digikey.se/product-detail/en/taiyo-yuden/GMK325BJ226MM-T/587-6141-1-ND/8619544" H 3600 3450 50  0001 C CNN "Distributor Link"
+F 6 "Taiyo Yuden" H 3600 3450 50  0001 C CNN "Manufacturer"
+F 7 "GMK325BJ226MM-T" H 3600 3450 50  0001 C CNN "Part Number"
 	1    3600 3450
 	-1   0    0    1
@@
 F 3 "~" H 4400 3450 50  0001 C CNN
 F 4 "35V" H 4150 3550 50  0000 L CNN "Voltage"
+F 5 "https://www.digikey.se/product-detail/en/murata-electronics/GRM319R6YA106KA12D/490-9964-1-ND/5026458" H 4400 3450 50  0001 C CNN "Distributor Link"
+F 6 "Murata Electronics" H 4400 3450 50  0001 C CNN "Manufacturer"
+F 7 "GRM319R6YA106KA12D" H 4400 3450 50  0001 C CNN "Part Number"
 	1    4400 3450
 	-1   0    0    1
@@
 F 3 "~" H 8300 3700 50  0001 C CNN
 F 4 "10V" H 8050 3800 50  0000 L CNN "Voltage"
+F 5 "https://www.digikey.se/product-detail/en/murata-electronics/GRM21BR61A226ME51L/490-10511-1-ND/5026441" H 8300 3700 50  0001 C CNN "Distributor Link"
+F 6 "Murata Electronics" H 8300 3700 50  0001 C CNN "Manufacturer"
+F 7 "GRM21BR61A226ME51L" H 8300 3700 50  0001 C CNN "Part Number"
 	1    8300 3700
 	-1   0    0    1
