File: TougherPowerMeter-FeatherWing.sch (KiCad schematic (older format))
At the start: 38 parts, among them J1 Jumper, J10 796639-2, J11 Jumper, J2 796639-2, J3 796639-2, J4 796639-2, J5 796639-2, J6 796639-2, J7 796639-2, J8 796639-2, J9 796639-2, U3 FeatherWing, U4 INA3221

Commit message: Add manufacturers, part numbers, and supplier links
Parts:
- C1, C18: Distributor Link (none) -> https://www.digikey.se/product-detail/en/kemet/C0603C475K9P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; Manufacturer (none) -> KEMET; Part Number (none) -> C0603C475K9PACTU; Voltage (none) -> 6.3V
- C8: Voltage (none) -> 50V
- D1: Distributor Link (none) -> https://www.digikey.se/product-detail/en/vishay-semiconduct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; Manufacturer (none) -> Vishay Semiconductor Diodes Division; Part Number (none) -> SMBJ16D-M3/I
- J10, J2, J3, J4, J5, J6, J7, J8, J9: Distributor Link (none) -> https://www.digikey.se/product-detail/en/te-connectivity-am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; Part Number (none) -> 796639-2
- R1, R10, R11, R12, R13, R14, R15, R2, R8, R9: Tolerance (none) -> 1%
- U4: Distributor Link (none) -> https://www.digikey.se/product-detail/en/texas-instruments/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; Manufacturer (none) -> Texas instruments; Part Number (none) -> INA3221AIRGV
Changed lines of the file:
@@
 F 2 "Package_DFN_QFN:Texas_RGV_S-PVQFN-N16_EP2.1x2.1mm" H 8300 3450 50  0001 C CNN
 F 3 "http://www.ti.com/lit/ds/symlink/ina3221.pdf" H 8300 3050 50  0001 C CNN
+F 4 "Texas instruments" H 8300 2350 50  0001 C CNN "Manufacturer"
+F 5 "INA3221AIRGV" H 8300 2350 50  0001 C CNN "Part Number"
+F 6 "https://www.digikey.se/product-detail/en/texas-instruments/INA3221AIRGVR/296-INA3221AIRGVRCT-ND/5143054" H 8300 2350 50  0001 C CNN "Distributor Link"
 	1    8300 2350
 	1    0    0    -1
@@
 F 2 "Capacitor_SMD:C_0603_1608Metric" H 7850 1250 50  0001 C CNN
 F 3 "~" H 7850 1250 50  0001 C CNN
+F 4 "50V" H 7850 1250 50  0001 C CNN "Voltage"
 	1    7850 1250
 	1    0    0    -1
@@
 F 2 "Resistor_SMD:R_0603_1608Metric" H 9100 1700 50  0001 C CNN
 F 3 "~" H 9100 1700 50  0001 C CNN
+F 4 "1%" H 9100 1700 50  0001 C CNN "Tolerance"
 	1    9100 1700
 	1    0    0    -1
@@
 F 2 "Resistor_SMD:R_0603_1608Metric" H 10000 1700 50  0001 C CNN
 F 3 "~" H 10000 1700 50  0001 C CNN
+F 4 "1%" H 10000 1700 50  0001 C CNN "Tolerance"
 	1    10000 1700
 	1    0    0    -1
@@
 F 2 "Resistor_SMD:R_0603_1608Metric" H 10300 1700 50  0001 C CNN
 F 3 "~" H 10300 1700 50  0001 C CNN
+F 4 "1%" H 10300 1700 50  0001 C CNN "Tolerance"
 	1    10300 1700
 	1    0    0    -1
@@
 F 2 "Resistor_SMD:R_0603_1608Metric" H 10600 1700 50  0001 C CNN
 F 3 "~" H 10600 1700 50  0001 C CNN
+F 4 "1%" H 10600 1700 50  0001 C CNN "Tolerance"
 	1    10600 1700
 	1    0    0    -1
@@
 F 3 "https://www.te.com/commerce/DocumentDelivery/DDEController?Action=srchrtrv&DocNm=796639&DocType=Customer+Drawing&DocLang=English" H 7900 4500 50  0001 C CNN
 F 4 "TE Connectivity" H 7900 4500 50  0001 C CNN "Manufacturer"
+F 5 "796639-2" H 7900 4500 50  0001 C CNN "Part Number"
+F 6 "https://www.digikey.se/product-detail/en/te-connectivity-amp-connectors/796639-2/A122654-ND/1130738" H 7900 4500 50  0001 C CNN "Distributor Link"
 	1    7900 4500
 	-1   0    0    -1
@@
 F 3 "https://www.te.com/commerce/DocumentDelivery/DDEController?Action=srchrtrv&DocNm=796639&DocType=Customer+Drawing&DocLang=English" H 7900 5250 50  0001 C CNN
 F 4 "TE Connectivity" H 7900 5250 50  0001 C CNN "Manufacturer"
+F 5 "796639-2" H 7900 5250 50  0001 C CNN "Part Number"
+F 6 "https://www.digikey.se/product-detail/en/te-connectivity-amp-connectors/796639-2/A122654-ND/1130738" H 7900 5250 50  0001 C CNN "Distributor Link"
 	1    7900 5250
 	-1   0    0    -1
@@
 F 3 "https://www.te.com/commerce/DocumentDelivery/DDEController?Action=srchrtrv&DocNm=796639&DocType=Customer+Drawing&DocLang=English" H 7900 6000 50  0001 C CNN
 F 4 "TE Connectivity" H 7900 6000 50  0001 C CNN "Manufacturer"
+F 5 "796639-2" H 7900 6000 50  0001 C CNN "Part Number"
+F 6 "https://www.digikey.se/product-detail/en/te-connectivity-amp-connectors/796639-2/A122654-ND/1130738" H 7900 6000 50  0001 C CNN "Distributor Link"
 	1    7900 6000
 	-1   0    0    -1
@@
 F 3 "https://www.te.com/commerce/DocumentDelivery/DDEController?Action=srchrtrv&DocNm=796639&DocType=Customer+Drawing&DocLang=English" H 8900 6000 50  0001 C CNN
 F 4 "TE Connectivity" H 8900 6000 50  0001 C CNN "Manufacturer"
+F 5 "796639-2" H 8900 6000 50  0001 C CNN "Part Number"
+F 6 "https://www.digikey.se/product-detail/en/te-connectivity-amp-connectors/796639-2/A122654-ND/1130738" H 8900 6000 50  0001 C CNN "Distributor Link"
 	1    8900 6000
 	-1   0    0    -1
@@
 F 3 "https://www.te.com/commerce/DocumentDelivery/DDEController?Action=srchrtrv&DocNm=796639&DocType=Customer+Drawing&DocLang=English" H 8900 5250 50  0001 C CNN
 F 4 "TE Connectivity" H 8900 5250 50  0001 C CNN "Manufacturer"
+F 5 "796639-2" H 8900 5250 50  0001 C CNN "Part Number"
+F 6 "https://www.digikey.se/product-detail/en/te-connectivity-amp-connectors/796639-2/A122654-ND/1130738" H 8900 5250 50  0001 C CNN "Distributor Link"
 	1    8900 5250
 	-1   0    0    -1
@@
 F 3 "https://www.te.com/commerce/DocumentDelivery/DDEController?Action=srchrtrv&DocNm=796639&DocType=Customer+Drawing&DocLang=English" H 8900 4500 50  0001 C CNN
 F 4 "TE Connectivity" H 8900 4500 50  0001 C CNN "Manufacturer"
+F 5 "796639-2" H 8900 4500 50  0001 C CNN "Part Number"
+F 6 "https://www.digikey.se/product-detail/en/te-connectivity-amp-connectors/796639-2/A122654-ND/1130738" H 8900 4500 50  0001 C CNN "Distributor Link"
 	1    8900 4500
 	-1   0    0    -1
@@
 F 3 "https://www.te.com/commerce/DocumentDelivery/DDEController?Action=srchrtrv&DocNm=796639&DocType=Customer+Drawing&DocLang=English" H 9900 4500 50  0001 C CNN
 F 4 "TE Connectivity" H 9900 4500 50  0001 C CNN "Manufacturer"
+F 5 "796639-2" H 9900 4500 50  0001 C CNN "Part Number"
+F 6 "https://www.digikey.se/product-detail/en/te-connectivity-amp-connectors/796639-2/A122654-ND/1130738" H 9900 4500 50  0001 C CNN "Distributor Link"
 	1    9900 4500
 	-1   0    0    -1
@@
 F 3 "https://www.te.com/commerce/DocumentDelivery/DDEController?Action=srchrtrv&DocNm=796639&DocType=Customer+Drawing&DocLang=English" H 9900 5250 50  0001 C CNN
 F 4 "TE Connectivity" H 9900 5250 50  0001 C CNN "Manufacturer"
+F 5 "796639-2" H 9900 5250 50  0001 C CNN "Part Number"
+F 6 "https://www.digikey.se/product-detail/en/te-connectivity-amp-connectors/796639-2/A122654-ND/1130738" H 9900 5250 50  0001 C CNN "Distributor Link"
 	1    9900 5250
 	-1   0    0    -1
@@
 F 3 "https://www.te.com/commerce/DocumentDelivery/DDEController?Action=srchrtrv&DocNm=796639&DocType=Customer+Drawing&DocLang=English" H 9900 6000 50  0001 C CNN
 F 4 "TE Connectivity" H 9900 6000 50  0001 C CNN "Manufacturer"
+F 5 "796639-2" H 9900 6000 50  0001 C CNN "Part Number"
+F 6 "https://www.digikey.se/product-detail/en/te-connectivity-amp-connectors/796639-2/A122654-ND/1130738" H 9900 6000 50  0001 C CNN "Distributor Link"
 	1    9900 6000
 	-1   0    0    -1
@@
 F 2 "Resistor_SMD:R_0603_1608Metric" H 10350 3150 50  0001 C CNN
 F 3 "~" H 10350 3150 50  0001 C CNN
+F 4 "1%" H 10350 3150 50  0001 C CNN "Tolerance"
 	1    10350 3150
 	1    0    0    -1
@@
 F 2 "Resistor_SMD:R_0603_1608Metric" H 10350 3700 50  0001 C CNN
 F 3 "~" H 10350 3700 50  0001 C CNN
+F 4 "1%" H 10350 3700 50  0001 C CNN "Tolerance"
 	1    10350 3700
 	1    0    0    -1
@@
 F 2 "Resistor_SMD:R_0603_1608Metric" H 9700 1700 50  0001 C CNN
 F 3 "~" H 9700 1700 50  0001 C CNN
+F 4 "1%" H 9700 1700 50  0001 C CNN "Tolerance"
 	1    9700 1700
 	1    0    0    -1
@@
 F 2 "Resistor_SMD:R_0603_1608Metric" H 9400 1700 50  0001 C CNN
 F 3 "~" H 9400 1700 50  0001 C CNN
+F 4 "1%" H 9400 1700 50  0001 C CNN "Tolerance"
 	1    9400 1700
 	1    0    0    -1
@@
 F 2 "Capacitor_SMD:C_0603_1608Metric" H 7450 1250 50  0001 C CNN
 F 3 "~" H 7450 1250 50  0001 C CNN
+F 4 "https://www.digikey.se/product-detail/en/kemet/C0603C475K9PACTU/399-3482-1-ND/754775" H 7450 1250 50  0001 C CNN "Distributor Link"
+F 5 "KEMET" H 7450 1250 50  0001 C CNN "Manufacturer"
+F 6 "C0603C475K9PACTU" H 7450 1250 50  0001 C CNN "Part Number"
+F 7 "6.3V" H 7450 1250 50  0001 C CNN "Voltage"
 	1    7450 1250
 	1    0    0    -1
@@
 F 2 "Resistor_SMD:R_0603_1608Metric" H 10350 2450 50  0001 C CNN
 F 3 "~" H 10350 2450 50  0001 C CNN
+F 4 "1%" H 10350 2450 50  0001 C CNN "Tolerance"
 	1    10350 2450
 	0    1    1    0
@@
 F 2 "Resistor_SMD:R_0603_1608Metric" H 10350 2550 50  0001 C CNN
 F 3 "~" H 10350 2550 50  0001 C CNN
+F 4 "1%" H 10350 2550 50  0001 C CNN "Tolerance"
 	1    10350 2550
 	0    1    1    0
@@
 F 2 "Diode_SMD:D_SMB" H 4900 5500 50  0001 C CNN
 F 3 "https://www.vishay.com/docs/87606/smbj5cdthrusmbj120cd.pdf" H 4850 5700 50  0001 C CNN
+F 4 "Vishay Semiconductor Diodes Division" V 4900 5700 50  0001 C CNN "Manufacturer"
+F 5 "SMBJ16D-M3/I" V 4900 5700 50  0001 C CNN "Part Number"
+F 6 "https://www.digikey.se/product-detail/en/vishay-semiconductor-diodes-division/SMBJ16D-M3-I/SMBJ16D-M3-IGICT-ND/9648416" V 4900 5700 50  0001 C CNN "Distributor Link"
 	1    4900 5700
 	0    1    1    0
@@
 F 2 "Capacitor_SMD:C_0603_1608Metric" H 2400 4200 50  0001 C CNN
 F 3 "~" H 2400 4200 50  0001 C CNN
+F 4 "https://www.digikey.se/product-detail/en/kemet/C0603C475K9PACTU/399-3482-1-ND/754775" H 2400 4200 50  0001 C CNN "Distributor Link"
+F 5 "KEMET" H 2400 4200 50  0001 C CNN "Manufacturer"
+F 6 "C0603C475K9PACTU" H 2400 4200 50  0001 C CNN "Part Number"
+F 7 "6.3V" H 2400 4200 50  0001 C CNN "Voltage"
 	1    2400 4200
 	1    0    0    -1

Commit message: Add submodule for the KiCad libraries.
Add submodule for the KiCad libraries and change
references to the libraries.
Parts:
- D1: symbol Diodes:SMBJxxxD -> Diode_BD:SMBJxxxD
Changed lines of the file:
@@
 	4900 5450 4900 5550
 $Comp
-L Diodes:SMBJxxxD D?
+L Diode_BD:SMBJxxxD D?
 U 1 1 5F6B0AA1
 P 4900 5700
